Commit message: Finished V1.0 by 2025.01

File: src/robot_description/urdf/robot.urdf (robot description, URDF)
Before this commit: robot robot_description, 8 links, 7 joints
Joints:
- joint joint1: limit lower=-3.1416 upper=3.1416 effort=49 velocity=3.14 -> lower=-2.9670 upper=2.9670 effort=49 velocity=3.14
- joint joint4: limit lower=-3.1416 upper=3.1416 effort=9 velocity=3.14 -> lower=-2.9670 upper=2.9670 effort=9 velocity=3.14
- joint joint6: limit lower=-3.1416 upper=3.1416 effort=9 velocity=3.14 -> lower=-2.9670 upper=2.9670 effort=9 velocity=3.14

File: src/robot_description/urdf/robot_gazebo.urdf (robot description, URDF)
Before this commit: robot robot_description, 7 links, 6 joints
Joints:
- joint joint1: limit lower=-3.1416 upper=3.1416 effort=49 velocity=3.14 -> lower=-2.9670 upper=2.9670 effort=49 velocity=3.14
- joint joint4: limit lower=-3.1416 upper=3.1416 effort=9 velocity=3.14 -> lower=-2.9670 upper=2.9670 effort=9 velocity=3.14
- joint joint6: limit lower=-3.1416 upper=3.1416 effort=9 velocity=3.14 -> lower=-2.9670 upper=2.9670 effort=9 velocity=3.14
