Commit message: Update the limit of arm380 by 20250403

File: src/robot_description/urdf/arm380.urdf (robot description, URDF)
Before this commit: robot arm380, 8 links, 7 joints
Joints:
- joint joint2: limit lower=-1.5708 upper=1.5708 effort=49 velocity=3.14 -> lower=-1.6232 upper=1.6232 effort=49 velocity=3.14
- joint joint3: limit lower=-1.5708 upper=1.5708 effort=49 velocity=3.14 -> lower=-2.6704 upper=2.6704 effort=49 velocity=3.14
- joint joint4: limit lower=-2.9670 upper=2.9670 effort=9 velocity=3.14 -> lower=-2.7576 upper=2.7576 effort=9 velocity=3.14
- joint joint5: limit lower=-1.5708 upper=1.5708 effort=9 velocity=3.14 -> lower=-1.5359 upper=1.5359 effort=9 velocity=3.14

File: src/robot_description/urdf/arm380_gazebo.urdf (robot description, URDF)
Before this commit: robot arm380, 8 links, 7 joints
Joints:
- joint joint2: limit lower=-1.5708 upper=1.5708 effort=49 velocity=3.14 -> lower=-1.6232 upper=1.6232 effort=49 velocity=3.14
- joint joint3: limit lower=-1.5708 upper=1.5708 effort=49 velocity=3.14 -> lower=-2.6704 upper=2.6704 effort=49 velocity=3.14
- joint joint4: limit lower=-2.9670 upper=2.9670 effort=9 velocity=3.14 -> lower=-2.7576 upper=2.7576 effort=9 velocity=3.14
- joint joint5: limit lower=-1.5708 upper=1.5708 effort=9 velocity=3.14 -> lower=-1.5359 upper=1.5359 effort=9 velocity=3.14

Commit message: Arm380 gazebo simulation finished by 20250403

File: src/robot_description/urdf/arm380.urdf (robot description, URDF)
Before this commit: robot arm380, 8 links, 7 joints
Joints:
- joint joint1: limit lower=-2.9670 upper=2.9670 effort=49 velocity=3.14 -> lower=-2.9670 upper=2.9670 effort=9 velocity=3.14
- joint joint2: limit lower=-1.6232 upper=1.6232 effort=49 velocity=3.14 -> lower=-1.6232 upper=1.6232 effort=9 velocity=3.14
- joint joint3: child 3_Link -> Link3; limit lower=-2.6704 upper=2.6704 effort=49 velocity=3.14 -> lower=-2.6704 upper=2.6704 effort=9 velocity=3.14; parent 2_link -> Link2
- joint joint4: limit lower=-2.7576 upper=2.7576 effort=9 velocity=3.14 -> lower=-2.7576 upper=2.7576 effort=3.3 velocity=3.14
- joint joint5: limit lower=-1.5359 upper=1.5359 effort=9 velocity=3.14 -> lower=-1.5359 upper=1.5359 effort=3.3 velocity=3.14
- joint joint6: limit lower=-2.9670 upper=2.9670 effort=9 velocity=3.14 -> lower=-2.9670 upper=2.9670 effort=3.3 velocity=3.14

File: src/robot_description/urdf/arm380_gazebo.urdf (robot description, URDF)
Before this commit: robot arm380, 8 links, 7 joints
Links:
- removed link world
Joints:
- removed joint base_joint
- joint joint1: limit lower=-2.9670 upper=2.9670 effort=49 velocity=3.14 -> lower=-2.9670 upper=2.9670 effort=9 velocity=3.14
- joint joint2: limit lower=-1.6232 upper=1.6232 effort=49 velocity=3.14 -> lower=-1.6232 upper=1.6232 effort=9 velocity=3.14
- joint joint3: child 3_Link -> Link3; limit lower=-2.6704 upper=2.6704 effort=49 velocity=3.14 -> lower=-2.6704 upper=2.6704 effort=9 velocity=3.14; parent 2_link -> Link2
- joint joint4: limit lower=-2.7576 upper=2.7576 effort=9 velocity=3.14 -> lower=-2.7576 upper=2.7576 effort=3.3 velocity=3.14
- joint joint5: limit lower=-1.5359 upper=1.5359 effort=9 velocity=3.14 -> lower=-1.5359 upper=1.5359 effort=3.3 velocity=3.14
- joint joint6: limit lower=-2.9670 upper=2.9670 effort=9 velocity=3.14 -> lower=-2.9670 upper=2.9670 effort=3.3 velocity=3.14

File: src/robot_gazebo/config/gazebo_arm380.urdf.xacro (robot description, xacro)
@@ -11,31 +11,30 @@
     <!-- 对一些link进行gazebo的属性设置 -->
     <gazebo reference="base_link">
-        <material>Gazebo/TurquoiseGlowOutline</material>
+        <material>Gazebo/Turquoise</material>
         <self_collide>false</self_collide>
         <gravity>false</gravity>
     </gazebo>
     <gazebo reference="Link1">
-        <material>Gazebo/TurquoiseGlowOutline</material>
-        <self_collide>false</self_collide>
+        <material>Gazebo/Turquoise</material>
         <gravity>false</gravity>
     </gazebo>
     <gazebo reference="Link2">
-        <material>Gazebo/TurquoiseGlowOutline</material>
+        <material>Gazebo/Turquoise</material>
         <gravity>false</gravity>
     </gazebo>
     <gazebo reference="Link3">
-        <material>Gazebo/TurquoiseGlowOutline</material>
+        <material>Gazebo/Turquoise</material>
         <gravity>false</gravity>
     </gazebo>
     <gazebo reference="Link4">
-        <material>Gazebo/TurquoiseGlowOutline</material>
+        <material>Gazebo/Turquoise</material>
         <gravity>false</gravity>
     </gazebo>
     <gazebo reference="Link5">
-        <material>Gazebo/TurquoiseGlowOutline</material>
+        <material>Gazebo/Turquoise</material>
         <gravity>false</gravity>
     </gazebo>
     <gazebo reference="Link6">
-        <material>Gazebo/TurquoiseGlowOutline</material>
+        <material>Gazebo/Turquoise</material>
         <gravity>false</gravity>
     </gazebo>

File: src/robot_gazebo/config/gazebo_arm620.urdf.xacro (robot description, xacro)
@@ -17,5 +17,4 @@
     <gazebo reference="Link1">
         <material>Gazebo/Turquoise</material>
-        <self_collide>false</self_collide>
         <gravity>false</gravity>
     </gazebo>
