Commit message: Add arm380 model by 20250403

File: src/robot_config/arm620_config/config/arm620.ros2_control.xacro (robot description, xacro)
@@ -1,5 +1,5 @@
 <?xml version="1.0"?>
 <robot xmlns:xacro="http://www.ros.org/wiki/xacro">
-    <xacro:macro name="robot_description_ros2_control" params="name initial_positions_file">
+    <xacro:macro name="arm620_ros2_control" params="name initial_positions_file">
         <xacro:property name="initial_positions" value="${load_yaml(initial_positions_file)['initial_positions']}"/>
         <ros2_control name="${name}" type="system">

File: src/robot_description/urdf/arm620_gazebo.urdf (robot description, URDF)
Before this commit: robot robot_description, 7 links, 6 joints
Links:
- link Link1: geometry collision mesh filename=file://$(find robot_description)/meshes/arm620/Link1.STL; visual mesh filename=file://$(find robot_description)/meshes/arm620/Link1.STL
- link Link2: geometry collision mesh filename=file://$(find robot_description)/meshes/arm620/Link2.STL; visual mesh filename=file://$(find robot_description)/meshes/arm620/Link2.STL
- link Link3: geometry collision mesh filename=file://$(find robot_description)/meshes/arm620/Link3.STL; visual mesh filename=file://$(find robot_description)/meshes/arm620/Link3.STL
- link Link4: geometry collision mesh filename=file://$(find robot_description)/meshes/arm620/Link4.STL; visual mesh filename=file://$(find robot_description)/meshes/arm620/Link4.STL
- link Link5: geometry collision mesh filename=file://$(find robot_description)/meshes/arm620/Link5.STL; visual mesh filename=file://$(find robot_description)/meshes/arm620/Link5.STL
- link Link6: geometry collision mesh filename=file://$(find robot_description)/meshes/arm620/Link6.STL; visual mesh filename=file://$(find robot_description)/meshes/arm620/Link6.STL
- link base_link: geometry collision mesh filename=file://$(find robot_description)/meshes/arm620/base_link.STL; visual mesh filename=file://$(find robot_description)/meshes/arm620/base_link.STL

File: src/robot_gazebo/config/gazebo_arm620.urdf.xacro (robot description, xacro)
@@ -1,4 +1,4 @@
 <?xml version="1.0"?>
-<robot xmlns:xacro="http://www.ros.org/wiki/xacro" name="robot_description">
+<robot xmlns:xacro="http://www.ros.org/wiki/xacro" name="arm620">
     <!-- Used for fixing robot to Gazebo 'base_link' 将机械手的基座固定在世界坐标上-->
     <link name="world"/>
@@ -8,33 +8,34 @@
     </joint>
     <!-- Import claw_description urdf file -->
-    <xacro:include filename="$(find robot_description)/urdf/robot_gazebo.urdf" />
+    <xacro:include filename="$(find robot_description)/urdf/arm620_gazebo.urdf" />
     <!-- 对一些link进行gazebo的属性设置 -->
     <gazebo reference="base_link">
+        <material>Gazebo/Turquoise</material>
         <self_collide>false</self_collide>
         <gravity>false</gravity>
     </gazebo>
-    <gazebo reference="link1">
-        <material>Gazebo/Purple</material>
+    <gazebo reference="Link1">
+        <material>Gazebo/Turquoise</material>
         <self_collide>false</self_collide>
         <gravity>false</gravity>
     </gazebo>
-    <gazebo reference="link2">
-        <material>Gazebo/Red</material>
+    <gazebo reference="Link2">
+        <material>Gazebo/Turquoise</material>
         <gravity>false</gravity>
     </gazebo>
-    <gazebo reference="link3">
-        <material>Gazebo/Blue</material>
+    <gazebo reference="Link3">
+        <material>Gazebo/Turquoise</material>
         <gravity>false</gravity>
     </gazebo>
-    <gazebo reference="link4">
-        <material>Gazebo/Green</material>
+    <gazebo reference="Link4">
+        <material>Gazebo/Turquoise</material>
         <gravity>false</gravity>
     </gazebo>
-    <gazebo reference="link5">
-        <material>Gazebo/Yellow</material>
+    <gazebo reference="Link5">
+        <material>Gazebo/Turquoise</material>
         <gravity>false</gravity>
     </gazebo>
-    <gazebo reference="link6">
-        <material>Gazebo/Orange</material>
+    <gazebo reference="Link6">
+        <material>Gazebo/Turquoise</material>
         <gravity>false</gravity>
     </gazebo>
@@ -94,5 +95,5 @@
     <gazebo>
         <plugin filename="libgazebo_ros2_control.so" name="gazebo_ros2_control">
-            <parameters>$(find robot_config)/config/ros2_controllers.yaml</parameters>
+            <parameters>$(find arm620_config)/config/ros2_controllers.yaml</parameters>
             <!-- <robot_param>robot_description</robot_param>
             <robot_param_node>robot_state_publisher</robot_param_node> -->
